File: DriveBoard_Hardware/DriveBoard_Hardware.sch (KiCad schematic (older format))
At the start: 12 parts, among them U1 TM4C129E_Launchpad, U2 MAX_3232, U3 OKI

Commit message: Completed board design
Parts:
- C1, C2, C3, C4, C5, C6: footprint Capacitors_SMD:C_0603_HandSoldering -> Capacitor_SMD:C_0603_1608Metric_Pad1.05x0.95mm_HandSolder
Changed lines of the file:
@@
 F 0 "C3" H 6275 2350 50  0000 L CNN
 F 1 "10uF" H 6275 2150 50  0000 L CNN
-F 2 "Capacitors_SMD:C_0603_HandSoldering" H 6288 2100 50  0001 C CNN
+F 2 "Capacitor_SMD:C_0603_1608Metric_Pad1.05x0.95mm_HandSolder" H 6288 2100 50  0001 C CNN
 F 3 "" H 6250 2250 50  0001 C CNN
 	1    6250 2250
@@
 F 0 "C6" H 7375 2350 50  0000 L CNN
 F 1 "10uF" H 7375 2150 50  0000 L CNN
-F 2 "Capacitors_SMD:C_0603_HandSoldering" H 7388 2100 50  0001 C CNN
+F 2 "Capacitor_SMD:C_0603_1608Metric_Pad1.05x0.95mm_HandSolder" H 7388 2100 50  0001 C CNN
 F 3 "" H 7350 2250 50  0001 C CNN
 	1    7350 2250
@@
 F 0 "C4" H 6910 3170 50  0000 L CNN
 F 1 ".1uF" H 6910 3020 50  0000 L CNN
-F 2 "Capacitors_SMD:C_0603_HandSoldering" H 6900 3100 50  0001 C CNN
+F 2 "Capacitor_SMD:C_0603_1608Metric_Pad1.05x0.95mm_HandSolder" H 6900 3100 50  0001 C CNN
 F 3 "" H 6900 3100 50  0001 C CNN
 	1    6900 3100
@@
 F 0 "C5" H 6910 3470 50  0000 L CNN
 F 1 ".1uF" H 6910 3320 50  0000 L CNN
-F 2 "Capacitors_SMD:C_0603_HandSoldering" H 6900 3400 50  0001 C CNN
+F 2 "Capacitor_SMD:C_0603_1608Metric_Pad1.05x0.95mm_HandSolder" H 6900 3400 50  0001 C CNN
 F 3 "" H 6900 3400 50  0001 C CNN
 	1    6900 3400
@@
 F 0 "C1" V 5500 3450 50  0000 L CNN
 F 1 ".1uF" V 5500 3200 50  0000 L CNN
-F 2 "Capacitors_SMD:C_0603_HandSoldering" H 5550 3400 50  0001 C CNN
+F 2 "Capacitor_SMD:C_0603_1608Metric_Pad1.05x0.95mm_HandSolder" H 5550 3400 50  0001 C CNN
 F 3 "" H 5550 3400 50  0001 C CNN
 	1    5550 3400
@@
 F 0 "C2" V 5600 3550 50  0000 L CNN
 F 1 ".1uF" V 5600 3300 50  0000 L CNN
-F 2 "Capacitors_SMD:C_0603_HandSoldering" H 5550 3500 50  0001 C CNN
+F 2 "Capacitor_SMD:C_0603_1608Metric_Pad1.05x0.95mm_HandSolder" H 5550 3500 50  0001 C CNN
 F 3 "" H 5550 3500 50  0001 C CNN
 	1    5550 3500

Commit message: Generated Gerbs and BOM
Other:
- note added: "Connectors"
- note removed: "Conectors"
Changed lines of the file:
@@
 Power Filtering
 Text Notes 7800 2800 0    98   ~ 20
-Conectors
+Connectors
 Wire Notes Line
 	5000 2650 8800 2650
