File: DriveBoard_Hardware/DriveBoard_Hardware.kicad_pcb (KiCad board)
At the start: 2 copper layers, 61 x 99.9 mm, 13 parts, among them U1 TM4C129E_Launchpad, U2 MAX_3232, U3 OKI

Commit message: add my name
Parts:
- added G***: LOGO, MRDT_ProjectLibary:SanfanLiu_sig21.8mmx12.3mm1, F.Cu at (158.2, 150.0)
