File: DriveBoard_Hardware/DriveBoard_Hardware.kicad_pcb (KiCad board)
At the start: 2 copper layers, 61 x 98 mm, 12 parts, among them U1 TM4C129E_Launchpad, U2 MAX_3232, U3 OKI

Commit message: Update
Small changes
Other:
- board text added: "Drive Board, R1 Mars Rover, 2019 Missouri S&T Andrew Simily"
Changed lines of the file:
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@@
   (general
     (thickness 1.6)
-    (drawings 20)
+    (drawings 21)
     (tracks 146)
     (zones 0)
@@
     (visible_elements 7FFFFFFF)
     (pcbplotparams
-      (layerselection 0x010fc_ffffffff)
+      (layerselection 0x0103c_ffffffff)
       (usegerberextensions false)
       (usegerberattributes false)
@@
       (outputformat 1)
       (mirror false)
-      (drillshape 1)
+      (drillshape 0)
       (scaleselection 1)
-      (outputdirectory ""))
+      (outputdirectory "gerbs/"))
   )
   (net 0 "")
@@
       (net 9 +5V))
   )
+  (gr_text "Drive Board, R1\nMars Rover, 2019\nMissouri S&T\nAndrew Simily" (at 121.412 133.35) (layer F.SilkS)
+    (effects (font (size 1.5 1.5) (thickness 0.3)) (justify left))
+  )
   (gr_text "Motor 2" (at 152.146 88.9 90) (layer F.SilkS)
