File: 2018Training/2018Training.kicad_pcb (KiCad board)
At the start: 2 copper layers, 61 x 100.1 mm, 14 parts, among them U1 TM4C129E_Launchpad, U2 OKI, U3 MAX_3232

Commit message: Revision 4, finished board
Parts:
- moved G*** 43.8 mm to (133.6, 96.5)
- moved Conn3 35.4 mm to (170.7, 86.1), turned to 270 degrees
Routing:
- net Net-(U1-PadGND): track 54.4 -> 0.00 mm
- net Net-(C2-Pad1): track 92.4 -> 43.1 mm, vias 5 -> 2
- net Net-(C1-Pad2): track 126.0 -> 98.0 mm
- net Net-(Conn2-Pad5): track 32.7 -> 19.0 mm, vias 0 -> 2
- net Net-(Conn2-Pad4): track 35.5 -> 23.6 mm, vias 0 -> 2
- net Net-(Conn3-Pad4): track 25.5 -> 18.1 mm, vias 0 -> 3
- net /Serial4: track 53.3 -> 50.9 mm
- net Net-(C5-Pad1): track 18.7 -> 20.0 mm
- net Net-(C3-Pad2): track 19.8 -> 20.8 mm
- net Net-(U1-PadPK1): track 52.5 -> 51.7 mm
- net Net-(Conn3-Pad5): track 19.8 -> 19.2 mm, vias 0 -> 2
- added copper zone on B.Cu, net Net-(C2-Pad1)
- added copper zone on F.Cu, net Net-(U1-PadGND)
