File: Driveboard_Hardware/Driveboard_Hardware.sch (KiCad schematic (older format))
At the start: 7 parts

Commit message: Layout
Parts:
- removed Conn?: Molex_SL_05, symbol MRDT_Connectors:Molex_SL_05
- removed U?: OKI, symbol MRDT_Devices:OKI
- added C1, C2, C3, C4, C5, C6: CP1_Small, Capacitor_SMD:C_0603_1608Metric_Pad1.05x0.95mm_HandSolder, symbol Device:CP1_Small
- added unit 1 of Conn1
- added Conn3: Molex_SL_05, MRDT_Connectors:MOLEX_SL_05_Horizontal, symbol MRDT_Connectors:Molex_SL_05
- added unit 3 of U1
- added unit 4 of U1
- added U2: OKI, MRDT_Devices:OKI_Horizontal, symbol MRDT_Devices:OKI
- Conn1: renamed from Conn?; footprint (none) -> MRDT_Connectors:Anderson_1_Horisontal
- Conn2: renamed from Conn?; footprint (none) -> MRDT_Connectors:MOLEX_SL_05_Horizontal
- U1: renamed from U?; footprint (none) -> MRDT_Shields:TM4C129E_Launchpad_X9
- U3: renamed from U?; footprint (none) -> MRDT_ICs:SOIC_16_3.9x9.9mm_Pitch1.27mm
Connections:
- net labels added: Earth
- net labels removed: GND
- wire segments 28 -> 57
- no-connect marks 0 -> 4
Other:
- moved on the sheet: Conn1C, Conn2, U3

Commit message: Board Revised and Checked
Parts:
- removed unit 3 of Conn1
- added unit 2 of Conn1
- C1, C2: value CP1_Small -> 10uF
- C3, C4, C5, C6: value CP1_Small -> .1uF
- Conn1: footprint MRDT_Connectors:Anderson_1_Horisontal -> MRDT_Connectors:Anderson_2_Horisontal_Side_by_Side
- Conn2: value Molex_SL_05 -> Motor1
- Conn3: value Molex_SL_05 -> Motor2
Changed lines of the file:
@@
 EESchema Schematic File Version 4
-LIBS:Driveboard_Hardware-cache
 EELAYER 26 0
 EELAYER END
@@
 P 6150 4400
 F 0 "Conn2" H 6277 4708 60  0000 L CNN
-F 1 "Molex_SL_05" H 6277 4602 60  0000 L CNN
+F 1 "Motor1" H 6277 4602 60  0000 L CNN
 F 2 "MRDT_Connectors:MOLEX_SL_05_Horizontal" H 6150 4400 60  0001 C CNN
 F 3 "" H 6150 4400 60  0001 C CNN
 	1    6150 4400
-	1    0    0    -1
-$EndComp
-$Comp
-L MRDT_Connectors:AndersonPP Conn1
-U 3 1 5BA5CBBA
-P 1750 2800
-F 0 "Conn1" H 1956 3187 60  0000 C CNN
-F 1 "AndersonPP" H 1956 3081 60  0000 C CNN
-F 2 "MRDT_Connectors:Anderson_1_Horisontal" H 1600 2250 60  0001 C CNN
-F 3 "" H 1600 2250 60  0001 C CNN
-	3    1750 2800
 	1    0    0    -1
 $EndComp
@@
 F 0 "Conn1" H 1956 3487 60  0000 C CNN
 F 1 "AndersonPP" H 1956 3381 60  0000 C CNN
-F 2 "MRDT_Connectors:Anderson_1_Horisontal" H 1600 2550 60  0001 C CNN
+F 2 "MRDT_Connectors:Anderson_2_Horisontal_Side_by_Side" H 1600 2550 60  0001 C CNN
 F 3 "" H 1600 2550 60  0001 C CNN
 	1    1750 3100
@@
 P 6150 4950
 F 0 "Conn3" H 6277 5258 60  0000 L CNN
-F 1 "Molex_SL_05" H 6277 5152 60  0000 L CNN
+F 1 "Motor2" H 6277 5152 60  0000 L CNN
 F 2 "MRDT_Connectors:MOLEX_SL_05_Horizontal" H 6150 4950 60  0001 C CNN
 F 3 "" H 6150 4950 60  0001 C CNN
@@
 Connection ~ 3400 2700
 Wire Wire Line
-	2150 2700 2400 2700
-Connection ~ 2400 2700
-Wire Wire Line
 	2150 3000 2400 3000
 Connection ~ 2400 3000
@@
 P 5300 3850
 F 0 "C5" H 5391 3896 50  0000 L CNN
-F 1 "CP1_Small" H 5391 3805 50  0000 L CNN
+F 1 ".1uF" H 5391 3805 50  0000 L CNN
 F 2 "Capacitor_SMD:C_0603_1608Metric_Pad1.05x0.95mm_HandSolder" H 5300 3850 50  0001 C CNN
 F 3 "~" H 5300 3850 50  0001 C CNN
@@
 P 2400 2850
 F 0 "C1" H 2491 2896 50  0000 L CNN
-F 1 "CP1_Small" H 2491 2805 50  0000 L CNN
+F 1 "10uF" H 2491 2805 50  0000 L CNN
 F 2 "Capacitor_SMD:C_0603_1608Metric_Pad1.05x0.95mm_HandSolder" H 2400 2850 50  0001 C CNN
 F 3 "~" H 2400 2850 50  0001 C CNN
@@
 P 5300 4150
 F 0 "C6" H 5391 4196 50  0000 L CNN
-F 1 "CP1_Small" H 5391 4105 50  0000 L CNN
+F 1 ".1uF" H 5391 4105 50  0000 L CNN
 F 2 "Capacitor_SMD:C_0603_1608Metric_Pad1.05x0.95mm_HandSolder" H 5300 4150 50  0001 C CNN
 F 3 "~" H 5300 4150 50  0001 C CNN
@@
 P 3950 4150
 F 0 "C3" H 4041 4196 50  0000 L CNN
-F 1 "CP1_Small" H 4041 4105 50  0000 L CNN
+F 1 ".1uF" H 4041 4105 50  0000 L CNN
 F 2 "Capacitor_SMD:C_0603_1608Metric_Pad1.05x0.95mm_HandSolder" H 3950 4150 50  0001 C CNN
 F 3 "~" H 3950 4150 50  0001 C CNN
@@
 P 3950 4250
 F 0 "C4" H 4041 4296 50  0000 L CNN
-F 1 "CP1_Small" H 4041 4205 50  0000 L CNN
+F 1 ".1uF" H 4041 4205 50  0000 L CNN
 F 2 "Capacitor_SMD:C_0603_1608Metric_Pad1.05x0.95mm_HandSolder" H 3950 4250 50  0001 C CNN
 F 3 "~" H 3950 4250 50  0001 C CNN
@@
 P 3400 2850
 F 0 "C2" H 3491 2896 50  0000 L CNN
-F 1 "CP1_Small" H 3491 2805 50  0000 L CNN
+F 1 "10uF" H 3491 2805 50  0000 L CNN
 F 2 "Capacitor_SMD:C_0603_1608Metric_Pad1.05x0.95mm_HandSolder" H 3400 2850 50  0001 C CNN
 F 3 "~" H 3400 2850 50  0001 C CNN
@@
 	1    0    0    -1
 $EndComp
+$Comp
+L MRDT_Connectors:AndersonPP Conn1
+U 2 1 5BB033AD
+P 1750 2800
+F 0 "Conn1" H 1956 3187 60  0000 C CNN
+F 1 "AndersonPP" H 1956 3081 60  0000 C CNN
+F 2 "MRDT_Connectors:Anderson_2_Horisontal_Side_by_Side" H 1600 2250 60  0001 C CNN
+F 3 "" H 1600 2250 60  0001 C CNN
+	2    1750 2800
+	1    0    0    -1
+$EndComp
+Wire Wire Line
+	2400 2700 2150 2700
+Connection ~ 2400 2700
 $EndSCHEMATC
